File: RobotPCB/Connectors.sch (KiCad schematic (older format))
At the start: 29 parts

Commit message: update
Parts:
- removed POWERPIN1, PSW1: Conn_01x02, symbol Connector_Generic:Conn_01x02
- added PW1: Conn_01x04, TerminalBlock:TerminalBlock_bornier-4_P5.08mm, symbol Connector_Generic:Conn_01x04
- D1: footprint (none) -> Diode_THT:D_DO-41_SOD81_P10.16mm_Horizontal
- DLED1, DLED2, DLED3: footprint (none) -> LED_SMD:LED_1206_3216Metric
- F1: footprint (none) -> Fuse:Fuse_Bourns_MF-RHT1000
- PA1: footprint (none) -> Connector_PinHeader_2.54mm:PinHeader_2x10_P2.54mm_Vertical
- PA2: footprint (none) -> Connector_PinHeader_2.54mm:PinHeader_2x03_P2.54mm_Vertical
- PM1, PM2, PM3, PM4, PM5, PM6, PM7, PM8: footprint (none) -> Connector_PinHeader_2.54mm:PinHeader_1x04_P2.54mm_Vertical
- PS1, PS2, PS3, PS4, PS5, PS6, PS7, PS8, PT1: footprint (none) -> Connector_PinHeader_2.54mm:PinHeader_1x03_P2.54mm_Vertical
- RLED1, RLED2, RLED3: footprint (none) -> Resistor_SMD:R_1206_3216Metric
Connections:
- net +12V: now also PW1.4 (Pin_4)
- net GND: now also PA1.11 (Pin_11), PA1.13 (Pin_13), PA1.15 (Pin_15), PA1.17 (Pin_17), PA1.19 (Pin_19), PA2.5 (Pin_5), PW1.1 (Pin_1); no longer PA1.10 (Pin_10), PA1.2 (Pin_2), PA1.4 (Pin_4), PA1.6 (Pin_6), PA1.8 (Pin_8), PA2.2 (Pin_2)
- net VCC: no longer PA2.5 (Pin_5), PA2.6 (Pin_6)
- net VDD: now also PA1.10 (Pin_10), PA1.2 (Pin_2), PA1.4 (Pin_4), PA1.6 (Pin_6), PA1.8 (Pin_8), PA2.2 (Pin_2), PA2.6 (Pin_6), PW1.3 (Pin_3); no longer PA1.11 (Pin_11), PA1.13 (Pin_13), PA1.15 (Pin_15), PA1.17 (Pin_17), PA1.19 (Pin_19)
- net at F1.2: now also PW1.2 (Pin_2)
