File: RobotPCB/Mega2560.sch (KiCad schematic (older format))
At the start: 1 part

Commit message: update
Parts:
- MEGA1: footprint aga:Mega2560Pro_Embed_RobotDyn -> Mega2560ProEmbed:Mega2560Pro_Embed_RobotDyn
Changed lines of the file:
@@
 F 0 "MEGA1" H 3450 5100 50  0000 C CNN
 F 1 "Mega2560Pro_Embed_RobotDyn" H 3500 5000 50  0000 C CNN
-F 2 "aga:Mega2560Pro_Embed_RobotDyn" H 3550 3350 50  0001 C CNN
+F 2 "Mega2560ProEmbed:Mega2560Pro_Embed_RobotDyn" H 3550 3350 50  0001 C CNN
 F 3 "" H 3500 3500 50  0001 C CNN
 	1    3550 3500
