File: RobotPCB/stepperMotors.sch (KiCad schematic (older format))
At the start: 40 parts, among them P1 Conn_02x03_Counter_Clockwise, P2 Conn_02x03_Counter_Clockwise, P3 Conn_02x03_Counter_Clockwise, P4 Conn_02x03_Counter_Clockwise, P5 Conn_02x03_Counter_Clockwise, P6 Conn_02x03_Counter_Clockwise, P7 Conn_02x03_Counter_Clockwise, P8 Conn_02x03_Counter_Clockwise, U1 A4988, U2 A4988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

Commit message: update
Parts:
- C1, C2, C3, C4, C5, C6, C7: footprint (none) -> Capacitor_SMD:CP_Elec_6.3x5.4
- C8: footprint (none) -> Capacitor_SMD:CP_Elec_6.3x5.4_Nichicon
- P1, P2, P3, P4, P5, P6, P7, P8: footprint (none) -> Connector_PinHeader_2.54mm:PinHeader_2x03_P2.54mm_Vertical
- R1, R10, R11, R12, R13, R14, R15, R16, R2, R3, R4, R5, R6, R7, R8, R9: footprint (none) -> Resistor_SMD:R_1206_3216Metric
Changed lines of the file:
@@
 F 0 "P1" H 1850 2450 50  0000 C CNN
 F 1 "Conn_02x03_Counter_Clockwise" H 1850 2876 50  0001 C CNN
-F 2 "" H 1800 2650 50  0001 C CNN
+F 2 "Connector_PinHeader_2.54mm:PinHeader_2x03_P2.54mm_Vertical" H 1800 2650 50  0001 C CNN
 F 3 "~" H 1800 2650 50  0001 C CNN
 	1    1800 2650
@@
 F 0 "R1" V 1550 2150 50  0000 C CNN
 F 1 "10K" V 1450 2150 50  0000 C CNN
-F 2 "" V 1380 2150 50  0001 C CNN
+F 2 "Resistor_SMD:R_1206_3216Metric" V 1380 2150 50  0001 C CNN
 F 3 "~" H 1450 2150 50  0001 C CNN
 	1    1450 2150
@@
 F 0 "C1" V 1700 1550 50  0000 R CNN
 F 1 "100uF" V 1400 1600 50  0000 R CNN
-F 2 "" H 1550 1500 50  0001 C CNN
+F 2 "Capacitor_SMD:CP_Elec_6.3x5.4" H 1550 1500 50  0001 C CNN
 F 3 "~" H 1550 1500 50  0001 C CNN
 	1    1550 1500
@@
 F 0 "P2" H 4500 2450 50  0000 C CNN
 F 1 "Conn_02x03_Counter_Clockwise" H 4500 2876 50  0001 C CNN
-F 2 "" H 4450 2650 50  0001 C CNN
+F 2 "Connector_PinHeader_2.54mm:PinHeader_2x03_P2.54mm_Vertical" H 4450 2650 50  0001 C CNN
 F 3 "~" H 4450 2650 50  0001 C CNN
 	1    4450 2650
@@
 F 0 "R2" V 4200 2150 50  0000 C CNN
 F 1 "10K" V 4100 2150 50  0000 C CNN
-F 2 "" V 4030 2150 50  0001 C CNN
+F 2 "Resistor_SMD:R_1206_3216Metric" V 4030 2150 50  0001 C CNN
 F 3 "~" H 4100 2150 50  0001 C CNN
 	1    4100 2150
@@
 F 0 "C2" V 4350 1550 50  0000 R CNN
 F 1 "100uF" V 4050 1600 50  0000 R CNN
-F 2 "" H 4200 1500 50  0001 C CNN
+F 2 "Capacitor_SMD:CP_Elec_6.3x5.4" H 4200 1500 50  0001 C CNN
 F 3 "~" H 4200 1500 50  0001 C CNN
 	1    4200 1500
@@
 F 0 "P3" H 7100 2450 50  0000 C CNN
 F 1 "Conn_02x03_Counter_Clockwise" H 7100 2876 50  0001 C CNN
-F 2 "" H 7050 2650 50  0001 C CNN
+F 2 "Connector_PinHeader_2.54mm:PinHeader_2x03_P2.54mm_Vertical" H 7050 2650 50  0001 C CNN
 F 3 "~" H 7050 2650 50  0001 C CNN
 	1    7050 2650
@@
 F 0 "R3" V 6800 2150 50  0000 C CNN
 F 1 "10K" V 6700 2150 50  0000 C CNN
-F 2 "" V 6630 2150 50  0001 C CNN
+F 2 "Resistor_SMD:R_1206_3216Metric" V 6630 2150 50  0001 C CNN
 F 3 "~" H 6700 2150 50  0001 C CNN
 	1    6700 2150
@@
 F 0 "C3" V 6950 1550 50  0000 R CNN
 F 1 "100uF" V 6650 1600 50  0000 R CNN
-F 2 "" H 6800 1500 50  0001 C CNN
+F 2 "Capacitor_SMD:CP_Elec_6.3x5.4" H 6800 1500 50  0001 C CNN
 F 3 "~" H 6800 1500 50  0001 C CNN
 	1    6800 1500
@@
 F 0 "P4" H 9650 2450 50  0000 C CNN
 F 1 "Conn_02x03_Counter_Clockwise" H 9650 2876 50  0001 C CNN
-F 2 "" H 9600 2650 50  0001 C CNN
+F 2 "Connector_PinHeader_2.54mm:PinHeader_2x03_P2.54mm_Vertical" H 9600 2650 50  0001 C CNN
 F 3 "~" H 9600 2650 50  0001 C CNN
 	1    9600 2650
@@
 F 0 "R4" V 9350 2150 50  0000 C CNN
 F 1 "10K" V 9250 2150 50  0000 C CNN
-F 2 "" V 9180 2150 50  0001 C CNN
+F 2 "Resistor_SMD:R_1206_3216Metric" V 9180 2150 50  0001 C CNN
 F 3 "~" H 9250 2150 50  0001 C CNN
 	1    9250 2150
@@
 F 0 "C4" V 9500 1550 50  0000 R CNN
 F 1 "100uF" V 9200 1600 50  0000 R CNN
-F 2 "" H 9350 1500 50  0001 C CNN
+F 2 "Capacitor_SMD:CP_Elec_6.3x5.4" H 9350 1500 50  0001 C CNN
 F 3 "~" H 9350 1500 50  0001 C CNN
 	1    9350 1500
@@
 F 0 "P5" H 1850 5000 50  0000 C CNN
 F 1 "Conn_02x03_Counter_Clockwise" H 1850 5426 50  0001 C CNN
-F 2 "" H 1800 5200 50  0001 C CNN
+F 2 "Connector_PinHeader_2.54mm:PinHeader_2x03_P2.54mm_Vertical" H 1800 5200 50  0001 C CNN
 F 3 "~" H 1800 5200 50  0001 C CNN
 	1    1800 5200
@@
 F 0 "R5" V 1550 4700 50  0000 C CNN
 F 1 "10K" V 1450 4700 50  0000 C CNN
-F 2 "" V 1380 4700 50  0001 C CNN
+F 2 "Resistor_SMD:R_1206_3216Metric" V 1380 4700 50  0001 C CNN
 F 3 "~" H 1450 4700 50  0001 C CNN
 	1    1450 4700
@@
 F 0 "C5" V 1700 4100 50  0000 R CNN
 F 1 "100uF" V 1400 4150 50  0000 R CNN
-F 2 "" H 1550 4050 50  0001 C CNN
+F 2 "Capacitor_SMD:CP_Elec_6.3x5.4" H 1550 4050 50  0001 C CNN
 F 3 "~" H 1550 4050 50  0001 C CNN
 	1    1550 4050
@@
 F 0 "P6" H 4500 5000 50  0000 C CNN
 F 1 "Conn_02x03_Counter_Clockwise" H 4500 5426 50  0001 C CNN
-F 2 "" H 4450 5200 50  0001 C CNN
+F 2 "Connector_PinHeader_2.54mm:PinHeader_2x03_P2.54mm_Vertical" H 4450 5200 50  0001 C CNN
 F 3 "~" H 4450 5200 50  0001 C CNN
 	1    4450 5200
@@
 F 0 "R6" V 4200 4700 50  0000 C CNN
 F 1 "10K" V 4100 4700 50  0000 C CNN
-F 2 "" V 4030 4700 50  0001 C CNN
+F 2 "Resistor_SMD:R_1206_3216Metric" V 4030 4700 50  0001 C CNN
 F 3 "~" H 4100 4700 50  0001 C CNN
 	1    4100 4700
@@
 F 0 "C6" V 4350 4100 50  0000 R CNN
 F 1 "100uF" V 4050 4150 50  0000 R CNN
-F 2 "" H 4200 4050 50  0001 C CNN
+F 2 "Capacitor_SMD:CP_Elec_6.3x5.4" H 4200 4050 50  0001 C CNN
 F 3 "~" H 4200 4050 50  0001 C CNN
 	1    4200 4050
@@
 F 0 "P7" H 7100 5000 50  0000 C CNN
 F 1 "Conn_02x03_Counter_Clockwise" H 7100 5426 50  0001 C CNN
-F 2 "" H 7050 5200 50  0001 C CNN
+F 2 "Connector_PinHeader_2.54mm:PinHeader_2x03_P2.54mm_Vertical" H 7050 5200 50  0001 C CNN
 F 3 "~" H 7050 5200 50  0001 C CNN
 	1    7050 5200
@@
 F 0 "R7" V 6800 4700 50  0000 C CNN
 F 1 "10K" V 6700 4700 50  0000 C CNN
-F 2 "" V 6630 4700 50  0001 C CNN
+F 2 "Resistor_SMD:R_1206_3216Metric" V 6630 4700 50  0001 C CNN
 F 3 "~" H 6700 4700 50  0001 C CNN
 	1    6700 4700
@@
 F 0 "C7" V 6950 4100 50  0000 R CNN
 F 1 "100uF" V 6650 4150 50  0000 R CNN
-F 2 "" H 6800 4050 50  0001 C CNN
+F 2 "Capacitor_SMD:CP_Elec_6.3x5.4" H 6800 4050 50  0001 C CNN
 F 3 "~" H 6800 4050 50  0001 C CNN
 	1    6800 4050
@@
 F 0 "P8" H 9650 5000 50  0000 C CNN
 F 1 "Conn_02x03_Counter_Clockwise" H 9650 5426 50  0001 C CNN
-F 2 "" H 9600 5200 50  0001 C CNN
+F 2 "Connector_PinHeader_2.54mm:PinHeader_2x03_P2.54mm_Vertical" H 9600 5200 50  0001 C CNN
 F 3 "~" H 9600 5200 50  0001 C CNN
 	1    9600 5200
@@
 F 0 "R8" V 9350 4700 50  0000 C CNN
 F 1 "10K" V 9250 4700 50  0000 C CNN
-F 2 "" V 9180 4700 50  0001 C CNN
+F 2 "Resistor_SMD:R_1206_3216Metric" V 9180 4700 50  0001 C CNN
 F 3 "~" H 9250 4700 50  0001 C CNN
 	1    9250 4700
@@
 F 0 "C8" V 9500 4100 50  0000 R CNN
 F 1 "100uF" V 9200 4150 50  0000 R CNN
-F 2 "" H 9350 4050 50  0001 C CNN
+F 2 "Capacitor_SMD:CP_Elec_6.3x5.4_Nichicon" H 9350 4050 50  0001 C CNN
 F 3 "~" H 9350 4050 50  0001 C CNN
 	1    9350 4050
@@
 F 0 "R9" V 1850 3000 50  0000 C CNN
 F 1 "100K" V 1750 3000 50  0000 C CNN
-F 2 "" V 1680 3000 50  0001 C CNN
+F 2 "Resistor_SMD:R_1206_3216Metric" V 1680 3000 50  0001 C CNN
 F 3 "~" H 1750 3000 50  0001 C CNN
 	1    1750 3000
@@
 F 0 "R10" V 4500 3000 50  0000 C CNN
 F 1 "100K" V 4400 3000 50  0000 C CNN
-F 2 "" V 4330 3000 50  0001 C CNN
+F 2 "Resistor_SMD:R_1206_3216Metric" V 4330 3000 50  0001 C CNN
 F 3 "~" H 4400 3000 50  0001 C CNN
 	1    4400 3000
@@
 F 0 "R11" V 7100 3000 50  0000 C CNN
 F 1 "100K" V 7000 3000 50  0000 C CNN
-F 2 "" V 6930 3000 50  0001 C CNN
+F 2 "Resistor_SMD:R_1206_3216Metric" V 6930 3000 50  0001 C CNN
 F 3 "~" H 7000 3000 50  0001 C CNN
 	1    7000 3000
@@
 F 0 "R12" V 9650 3000 50  0000 C CNN
 F 1 "100K" V 9550 3000 50  0000 C CNN
-F 2 "" V 9480 3000 50  0001 C CNN
+F 2 "Resistor_SMD:R_1206_3216Metric" V 9480 3000 50  0001 C CNN
 F 3 "~" H 9550 3000 50  0001 C CNN
 	1    9550 3000
@@
 F 0 "R13" V 1850 5550 50  0000 C CNN
 F 1 "100K" V 1750 5550 50  0000 C CNN
-F 2 "" V 1680 5550 50  0001 C CNN
+F 2 "Resistor_SMD:R_1206_3216Metric" V 1680 5550 50  0001 C CNN
 F 3 "~" H 1750 5550 50  0001 C CNN
 	1    1750 5550
@@
 F 0 "R14" V 4500 5550 50  0000 C CNN
 F 1 "100K" V 4400 5550 50  0000 C CNN
-F 2 "" V 4330 5550 50  0001 C CNN
+F 2 "Resistor_SMD:R_1206_3216Metric" V 4330 5550 50  0001 C CNN
 F 3 "~" H 4400 5550 50  0001 C CNN
 	1    4400 5550
@@
 F 0 "R15" V 7100 5550 50  0000 C CNN
 F 1 "100K" V 7000 5550 50  0000 C CNN
-F 2 "" V 6930 5550 50  0001 C CNN
+F 2 "Resistor_SMD:R_1206_3216Metric" V 6930 5550 50  0001 C CNN
 F 3 "~" H 7000 5550 50  0001 C CNN
 	1    7000 5550
@@
 F 0 "R16" V 9650 5550 50  0000 C CNN
 F 1 "100K" V 9550 5550 50  0000 C CNN
-F 2 "" V 9480 5550 50  0001 C CNN
+F 2 "Resistor_SMD:R_1206_3216Metric" V 9480 5550 50  0001 C CNN
 F 3 "~" H 9550 5550 50  0001 C CNN
 	1    9550 5550
